Commit message: hokuyo added

File: src/hydrone_aerial_description/urdf/hydrone.xacro (robot description, xacro)
@@ -196,5 +196,5 @@
       <origin xyz="0 0 0.0" rpy="0 0 0"/>
       <geometry>
-        <mesh filename="package://hydrone_aerial_description/meshes/lds.stl" scale="0.001 0.001 0.001"/>
+        <mesh filename="package://hydrone_aerial_description/meshes/lds.stl" scale="1.0 1.0 1.0"/>
       </geometry>
       <material name="dark"/>
